File: bmc-breakout-board.sch (KiCad schematic (older format))
At the start: 49 parts, among them J1 PinHeader_2x4, J10 PinHeader_2x4, J11 PinHeader_2x05, J12 61300411121, J13 0473460001, J14 PCIE_BUS_x1, J15 0473460001, J16 PinHeader_1x07, J17 UE27AC54100, J2 PinHeader_2x13, J3 PinHeader_2x08, J4 61300411121, J5 ME1016813401101, J6 61300411121, J7 DC_SOCKET, J8 PinHeader_2x05, J9 PinHeader_1x07, Q1 SI2337DS, U1 FT234XD-R

Commit message: Introduce schematic sheets
Parts:
- removed C1, C2, C3, C4, C5, C7: C_100n_0402, bmc-breakout-board-footprints:0402-cap, symbol bmc-breakout-board:C_100n_0402
- removed C10: C_10u_25V_0603, bmc-breakout-board-footprints:0603-cap, symbol bmc-breakout-board:C_10u_25V_0603
- removed C11, C9: C_100n_0402_16V, bmc-breakout-board-footprints:0402-cap, symbol bmc-breakout-board:C_100n_0402_16V
- removed C12, C8: C_1n_0603, bmc-breakout-board-footprints:0603-cap, symbol bmc-breakout-board:C_1n_0603
- removed C6: C_1u_0402, bmc-breakout-board-footprints:0402-cap, symbol bmc-breakout-board:C_1u_0402
- removed D1, D2, D3: TPD2E009, bmc-breakout-board-footprints:SOT-3, symbol bmc-breakout-board:TPD2E009
- removed J1, J10: PinHeader_2x4, bmc-breakout-board-footprints:PinHeader_2x04_P2.54mm_Vertical, symbol bmc-breakout-board:PinHeader_2x4
- removed J11, J8: PinHeader_2x05, bmc-breakout-board-footprints:PinHeader_2x05_P2.54mm_Vertical, symbol bmc-breakout-board:PinHeader_2x05
- removed J12, J4, J6: 61300411121, bmc-breakout-board-footprints:PinHeader_1x4_P2.54mm_Drill1.02mm, symbol bmc-breakout-board:61300411121
- removed J13, J15: 0473460001, bmc-breakout-board-footprints:USB_Micro_B_Female_0473460001, symbol bmc-breakout-board:0473460001
- removed J14: PCIE_BUS_x1, bmc-breakout-board-footprints:BUS_PCIexpress_x1, symbol bmc-breakout-board:PCIE_BUS_x1
- removed J16, J9: PinHeader_1x07, bmc-breakout-board-footprints:PinHeader_1x07_P2.54mm_Vertical, symbol bmc-breakout-board:PinHeader_1x07
- removed J17: UE27AC54100, bmc-breakout-board-footprints:USB_A_Female_UE27AC54100, symbol bmc-breakout-board:UE27AC54100
- removed J2: PinHeader_2x13, bmc-breakout-board-footprints:PinHeader_2x13_P2.54mm_Vertical, symbol bmc-breakout-board:PinHeader_2x13
- removed J3: PinHeader_2x08, bmc-breakout-board-footprints:PinHeader_2x08_P2.54mm_Vertical, symbol bmc-breakout-board:PinHeader_2x08
- removed J5: ME1016813401101, bmc-breakout-board-footprints:ME1016813401101, symbol bmc-breakout-board:ME1016813401101
- removed J7: DC_SOCKET, bmc-breakout-board-footprints:DC_SOCKET, symbol bmc-breakout-board:DC_SOCKET
- removed L1: 744235900, bmc-breakout-board-footprints:744235900, symbol bmc-breakout-board:744235900
- removed Q1: SI2337DS, bmc-breakout-board-footprints:SOT-23-3, symbol bmc-breakout-board:SI2337DS
- removed R1: R_0R_0402, bmc-breakout-board-footprints:0402-res, symbol bmc-breakout-board:R_0R_0402
- removed R2: R_10k_0402, bmc-breakout-board-footprints:0402-res, symbol bmc-breakout-board:R_10k_0402
- removed R3, R6: R_220R_0402, bmc-breakout-board-footprints:0402-res, symbol bmc-breakout-board:R_220R_0402
- removed R4, R5: R_22R_0402, bmc-breakout-board-footprints:0402-res, symbol bmc-breakout-board:R_22R_0402
- removed S1: EG1218, bmc-breakout-board-footprints:Switch_Slide_11.6x4mm_EG1218, symbol bmc-breakout-board:EG1218
- removed U1: FT234XD-R, bmc-breakout-board-footprints:DFN-12-1EP_3x3mm, symbol bmc-breakout-board:FT234XD-R
Connections:
- no-connect marks 17 -> 0
Other:
- note added: "Data Center Secure Control Module (DC-SCM) Breakout Board"
- note added: "Logotypes"
- note added: "Mechanical"
- note removed: "12VDC IN"
- note removed: "Edge connector"
- note removed: "GND probes"
- note removed: "Power filtering"
- moved on the sheet: MP1, MP2, MP3, N1, N2, TP1, TP2
