File: sensors.kicad_sch (KiCad schematic)
At the start: 0 parts

Commit message: [#92504] Add temperature sensor
Parts:
- added C5: C_100n_0402, antmicro-footprints:C_0402_1005Metric, symbol antmicroCapacitors0402:C_100n_0402
- added R2, R4, R5: R_4k7_0402, antmicro-footprints:R_0402_1005Metric, symbol antmicroResistors0402:R_4k7_0402
- added U1: TMP75AIDR, antmicro-footprints:SOIC-8_3.9x4.9x1.75mm_P1.27mm, symbol antmicroTemperatureSensorsAnalogandDigitalOutput:TMP75AIDR
Connections:
- new net: R5.1, U1.3 (ALERT)
- new net +3V3: C5.2, R2.2, R4.2, R5.2, U1.8 (V+)
- new net DC_SCM_I2C6.SCL: R2.1, U1.2 (SCL)
- new net DC_SCM_I2C6.SDA: R4.1, U1.1 (SDA)
- new net GND: C5.1, U1.4 (GND), U1.5 (A2), U1.6 (A1), U1.7 (A0)
Other:
- note added: "TEMPERATURE SENSOR"
