File: usbs.kicad_sch (KiCad schematic)
At the start: 34 parts, among them J2 USB-A_Amphenol_UE27AC54100, J3 USB-C_GCT_USB4105-GF-A, J4 USB-C_GCT_USB4105-GF-A, U12 FT4232H_VQFN, Y1 Resonator_12MHz_ABM8G

Commit message: [#92504] Connect FT4232H QSPI
Parts:
- removed U12: FT4232H_VQFN, antmicro-footprints:QFN-56-1EP_8x8mm_P0.5mm, symbol antmicroInterfaceControllers:FT4232H_VQFN
- added U3: FT4232H_VQFN, antmicro-footprints:QFN-56-1EP_8x8mm_P0.5mm, symbol antmicroInterfaceControllers:FT4232H_VQFN
Connections:
- net +3V3: now also U3.16 (V_{CCIO}), U3.36 (V_{CCIO}), U3.44 (V_{REGIN}), U3.50 (V_{CCIO})
- net DC_SCM_QSPI.IO0: now also U3.13 (ADBUS1)
- net DC_SCM_QSPI.IO1: now also U3.14 (ADBUS2)
- net DC_SCM_QSPI.IO2: now also U3.18 (ADBUS5)
- net DC_SCM_QSPI.IO3: now also U3.19 (ADBUS6)
- net DC_SCM_QSPI.SCK: now also U3.12 (ADBUS0)
- net DC_SCM_QSPI.~{CS0}: now also U3.15 (ADBUS3)
- net DC_SCM_QSPI.~{CS1}: now also U3.17 (ADBUS4)
- net GND: now also U3.10 (TEST), U3.21 (GND), U3.41 (GND), U3.45 (GND), U3.57 (GND)
- net VCORE: now also U3.2 (V_{CORE}), U3.31 (V_{CORE}), U3.43 (V_{REGOUT})
- net VPHY: now also U3.5 (V_{PHY})
- net VPLL: now also U3.9 (V_{PLL})
- net XI: now also U3.3 (OSCI)
- net XO: now also U3.4 (OSCO)
- net at R33.1: now also U3.33 (CDBUS1)
- net at R34.2: now also U3.11 (~{RESET})
- net at R32.1: now also U3.32 (CDBUS0)
- net at R26.2: now also U3.6 (REF)
- net at R39.2: now also U3.7 (D-)
- net at R38.2: now also U3.8 (D+)
- no-connect marks 31 -> 32
