File: jtag.kicad_sch (KiCad schematic)
At the start: 2 parts, among them J8 PinHeader_1x2_P1.27mm_Drill0.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, J9 PinHeader_2x5_P1.27mm_SMD_Shr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

Commit message: [#93514] Propagate title and date across all of the sheets
Other:
- title: (none) -> Datacenter Secure Control Module Breakout Board
Changed lines of the file:
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@@
 	(generator_version "9.0")
 	(paper "A3")
+	(title_block
+		(title "Datacenter Secure Control Module Breakout Board")
+		(date "2021-12-16")
+		(rev "2.0.0")
+	)
 	(text "JTAG\n"
 		(exclude_from_sim no)
