File: led.kicad_sch (KiCad schematic)
At the start: 6 parts

Commit message: [#93514] Propagate title and date across all of the sheets
Other:
- title: (none) -> Datacenter Secure Control Module Breakout Board
Changed lines of the file:
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@@
 	(generator_version "9.0")
 	(paper "A3")
+	(title_block
+		(title "Datacenter Secure Control Module Breakout Board")
+		(date "2021-12-16")
+		(rev "2.0.0")
+	)
 	(text "Indicator LEDs"
 		(exclude_from_sim no)
