File: bmc-breakout-board.kicad_sch (KiCad schematic)
At the start: 14 parts

Commit message: [#93949] Change Logo to be on copper layer
Parts:
- N1: footprint antmicro-footprints:antmicro-logo_scaled_20mm_mask -> antmicro-footprints:antmicro-logo_scaled_20mm
- N2: footprint antmicro-footprints:OSHW-Logo_5.7x6mm_Mask -> antmicro-footprints:OSHW-Logo_5.7x6mm_Copper
Changed lines of the file:
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@@
 			)
 		)
-		(property "Footprint" "antmicro-footprints:antmicro-logo_scaled_20mm_mask"
+		(property "Footprint" "antmicro-footprints:antmicro-logo_scaled_20mm"
 			(at 264.16 231.14 0)
 			(effects
@@
 			)
 		)
-		(property "Footprint" "antmicro-footprints:OSHW-Logo_5.7x6mm_Mask"
+		(property "Footprint" "antmicro-footprints:OSHW-Logo_5.7x6mm_Copper"
 			(at 331.978 196.596 0)
 			(effects

Commit message: [#93949] Update oshw logo to copper+mask
Parts:
- N2: footprint antmicro-footprints:OSHW-Logo_5.7x6mm_Copper -> antmicro-footprints:oshw-logo
Changed lines of the file:
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@@
 			)
 		)
-		(property "Footprint" "antmicro-footprints:OSHW-Logo_5.7x6mm_Copper"
+		(property "Footprint" "antmicro-footprints:oshw-logo"
 			(at 331.978 196.596 0)
 			(effects
